Commit message: add launch, param for localization, navigation

File: description/gazebo_control.xacro (robot description, xacro)
@@ -6,8 +6,8 @@
             <left_joint>left_wheel_joint</left_joint>
             <right_joint>right_wheel_joint</right_joint>
-            <wheel_separation>0.35</wheel_separation>
-            <wheel_diameter>0.1</wheel_diameter>
+            <wheel_separation>0.2</wheel_separation>
+            <wheel_diameter>0.03</wheel_diameter>
             <!-- Limits -->
-            <max_wheel_torque>1000</max_wheel_torque>
+            <max_wheel_torque>500</max_wheel_torque>
             <max_wheel_acceleration>10.0</max_wheel_acceleration>
             <!-- Output -->

File: description/lidar.xacro (robot description, xacro)
@@ -4,7 +4,7 @@
 	<xacro:include filename="colours.xacro"/> -->
 	<joint name="laser_joint" type="fixed">
-		<parent link="front_caster_wheel"/>
+		<parent link="chassis"/>
 		<child link="laser_frame"/>
-		<origin xyz="0 0 ${chassis_height + 0.01}"/>
+		<origin xyz="${(chassis_length/2)-0.05} 0 ${(chassis_height/2) + 0.01}"/>
 	</joint>
 	<link name="laser_frame">
@@ -36,5 +36,5 @@
 			<pose> 0 0 0 0 0 0 </pose>
 			<visualize>true</visualize>
-			<update_rate>5.5</update_rate>
+			<update_rate>10.0</update_rate>
 			<ray>
 				<scan>

File: description/robot_core.xacro (robot description, xacro)
@@ -21,4 +21,5 @@
 	<xacro:property name="caster_wheel_origin_y" value="0.0"/>
 	<xacro:property name="caster_wheel_origin_z" value="${wheel_origin_z}"/>
+	<xacro:property name="mu" value="0.001"/>
 <!-- BASE LINK-->
 	<link name="base_link">
@@ -29,4 +30,12 @@
 		<origin xyz="${chassis_origin_x} ${chassis_origin_y} ${chassis_origin_z}"/>
 	</joint>
+    <!-- BASE_FOOTPRINT LINK -->
+    <joint name="base_footprint_joint" type="fixed">
+        <parent link="base_link"/>
+        <child link="base_footprint"/>
+        <origin xyz="0 0 0" rpy="0 0 0"/>
+    </joint>
+    <link name="base_footprint">
+    </link>
 <!-- CHASSIS-->
 	<link name="chassis">
@@ -128,6 +137,6 @@
 	<gazebo reference="front_caster_wheel">
 		<material>Gazebo/White</material>
-		<mu1 value="0.001"/>
-		<mu2 value="0.001"/>
+		<mu1 value="${mu}"/>
+		<mu2 value="${mu}"/>
 	</gazebo>
 <!-- BACK CASTER WHEEL-->
@@ -156,6 +165,6 @@
 	<gazebo reference="back_caster_wheel">
 		<material>Gazebo/White</material>
-		<mu1 value="0.001"/>
-		<mu2 value="0.001"/>
+		<mu1 value="${mu}"/>
+		<mu2 value="${mu}"/>
 	</gazebo>
 </robot>

Commit message: real robot sync

File: description/gazebo_control.xacro (robot description, xacro)
@@ -6,6 +6,6 @@
             <left_joint>left_wheel_joint</left_joint>
             <right_joint>right_wheel_joint</right_joint>
-            <wheel_separation>0.2</wheel_separation>
-            <wheel_diameter>0.03</wheel_diameter>
+            <wheel_separation>0.345</wheel_separation>
+            <wheel_diameter>0.1</wheel_diameter>
             <!-- Limits -->
             <max_wheel_torque>500</max_wheel_torque>

File: description/robot.urdf.xacro (robot description, xacro)
@@ -4,9 +4,4 @@
 	<xacro:include filename="robot_core.xacro" />
 	<xacro:include filename="lidar.xacro"/>
-	<xacro:if value="$(arg use_ros2_control)">
-		<xacro:include filename="ros2_control.xacro"/>
-	</xacro:if>
-	<xacro:unless value="$(arg use_ros2_control)">
-		<xacro:include filename="gazebo_control.xacro"/>
-	</xacro:unless>
+	<xacro:include filename="ros2_control.xacro"/>
 </robot>

File: description/robot_core.xacro (robot description, xacro)
@@ -3,16 +3,16 @@
 	<xacro:include filename="colours.xacro"/>
 	<xacro:include filename="inertial_macros.xacro"/>
-    <xacro:property name="chassis_length" value="0.3"/>
-    <xacro:property name="chassis_width" value="0.2"/>
-    <xacro:property name="chassis_height" value="0.11"/>
+    <xacro:property name="chassis_length" value="0.330"/>
+    <xacro:property name="chassis_width" value="0.315"/>
+    <xacro:property name="chassis_height" value="0.2"/>
     <xacro:property name="chassis_mass" value="1.0"/>
 	<xacro:property name="chassis_origin_x" value="${(chassis_length/2) + 0.005}"/>
 	<xacro:property name="chassis_origin_y" value="0.0"/>
 	<xacro:property name="chassis_origin_z" value="${(chassis_height/2 + wheel_radius)}"/>
-    <xacro:property name="wheel_radius" value="0.03"/>
-    <xacro:property name="wheel_thickness" value="0.015"/>
+    <xacro:property name="wheel_radius" value="0.05"/>
+    <xacro:property name="wheel_thickness" value="0.03"/>
     <xacro:property name="wheel_mass" value="0.05"/>
 	<xacro:property name="wheel_origin_x" value="0.0"/>
-	<xacro:property name="wheel_origin_y" value="${(chassis_width/2) + (wheel_thickness/2) + 0.01}"/>
+	<xacro:property name="wheel_origin_y" value="${(chassis_width/2) + (wheel_thickness/2)}"/>
 	<xacro:property name="wheel_origin_z" value="${chassis_height/2}"/>
     <xacro:property name="caster_wheel_radius" value="${wheel_radius}"/>
@@ -168,3 +168,26 @@
 		<mu2 value="${mu}"/>
 	</gazebo>
+	<joint name="back_frame_joint" type="fixed">
+		<parent link="chassis"/>
+		<child link="back_frame"/>
+		<origin xyz="-${chassis_length/4} 0 ${chassis_height/2}" rpy="0 0 0"/>
+	</joint>
+	<link name="back_frame">
+		<visual>
+			<origin xyz="0 0 ${chassis_height/2}" rpy="0 0 0"/>
+			<geometry>
+				<box size="${chassis_length/2} ${chassis_width} ${chassis_height}"/>
+			</geometry>
+			<material name="orange"/>
+		</visual>
+		<collision>
+			<origin xyz="0 0 ${chassis_height/2}" rpy="0 0 0"/>
+			<geometry>
+				<box size="${chassis_length/2} ${chassis_width} ${chassis_height/2}"/>
+			</geometry>
+		</collision>
+		<xacro:inertial_box mass="${chassis_mass/2}" x="${chassis_length/2}" y="${chassis_width}" z="${chassis_height/2}">
+			<origin xyz="0 0 0" rpy="0 0 0"/>
+		</xacro:inertial_box>
+	</link>
 </robot>

File: description/ros2_control.xacro (robot description, xacro)
@@ -2,4 +2,31 @@
 <robot xmlns:xacro="http://www.ros.org/wiki/xacro">
 <!--ROS2_CONTROL-->
+	<!-- <ros2_control name="RealRobot" type="system">
+		<hardware>
+			<plugin>diffdrive_arduino/DiffDriveArduino</plugin>
+			<param name="left_wheel_name">left_wheel_joint</param>
+			<param name="right_wheel_name">right_wheel_joint</param>
+			<param name="loop_rate">20</param>
+			<param name="device">/dev/serial/by-path/pci-0000:05:00.3-usb-0:2:1.0-port0</param>
+			<param name="baud_rate">115200</param>
+			<param name="timeout">100</param>
+		</hardware>
+		<joint name="left_wheel_joint">
+			<command_interface name="velocity">
+				<param name="min">-0.5</param>
+				<param name="max">0.5</param>
+			</command_interface>
+			<state_interface name="velocity"/>
+			<state_interface name="position"/>
+		</joint>
+		<joint name="right_wheel_joint">
+			<command_interface name="velocity">
+				<param name="min">-0.5</param>
+				<param name="max">0.5</param>
+			</command_interface>
+			<state_interface name="velocity"/>
+			<state_interface name="position"/>
+		</joint>
+	</ros2_control> -->
 	<ros2_control name="GazeboSystem" type="system">
 		<hardware>
@@ -8,6 +35,6 @@
 		<joint name="left_wheel_joint">
 			<command_interface name="velocity">
-				<param name="min">-10</param>
-				<param name="max">10</param>
+				<param name="min">-1.0</param>
+				<param name="max">1.0</param>
 			</command_interface>
 			<state_interface name="position"/>
@@ -16,6 +43,6 @@
 		<joint name="right_wheel_joint">
 			<command_interface name="velocity">
-				<param name="min">-10</param>
-				<param name="max">10</param>
+				<param name="min">-1.0</param>
+				<param name="max">1.0</param>
 			</command_interface>
 			<state_interface name="position"/>
