Commit message: change robot orientation with respect to right hand rule

File: description/robot_core.xacro (robot description, xacro)
@@ -7,23 +7,17 @@
     <xacro:property name="chassis_height" value="0.11"/>
     <xacro:property name="chassis_mass" value="1.0"/>
-	<xacro:property name="chassis_origin_x" value="0.0"/>
-	<xacro:property name="chassis_origin_y" value="${(chassis_length/2) + 0.05}"/>
+	<xacro:property name="chassis_origin_x" value="${(chassis_length/2) + 0.005}"/>
+	<xacro:property name="chassis_origin_y" value="0.0"/>
 	<xacro:property name="chassis_origin_z" value="${(chassis_height/2 + wheel_radius)}"/>
     <xacro:property name="wheel_radius" value="0.03"/>
-    <xacro:property name="wheel_thickness" value="0.03"/>
+    <xacro:property name="wheel_thickness" value="0.015"/>
     <xacro:property name="wheel_mass" value="0.05"/>
-    <xacro:property name="wheel_offset_x" value="0.0"/>
-    <xacro:property name="wheel_offset_y" value="0.0"/>
-    <xacro:property name="wheel_offset_z" value="0.0"/>
-	<xacro:property name="wheel_origin_x" value="${(chassis_width/2) + (wheel_thickness/2) + 0.01}"/>
-	<xacro:property name="wheel_origin_y" value="0.0"/>
+	<xacro:property name="wheel_origin_x" value="0.0"/>
+	<xacro:property name="wheel_origin_y" value="${(chassis_width/2) + (wheel_thickness/2) + 0.01}"/>
 	<xacro:property name="wheel_origin_z" value="${chassis_height/2}"/>
     <xacro:property name="caster_wheel_radius" value="${wheel_radius}"/>
     <xacro:property name="caster_wheel_mass" value="0.01"/>
-	<xacro:property name="caster_wheel_offset_x" value="0.0"/>
-    <xacro:property name="caster_wheel_offset_y" value="0.0"/>
-    <xacro:property name="caster_wheel_offset_z" value="0.0"/>
-	<xacro:property name="caster_wheel_origin_x" value="0.0"/>
-	<xacro:property name="caster_wheel_origin_y" value="${(chassis_length/2)-caster_wheel_radius}"/>
+	<xacro:property name="caster_wheel_origin_x" value="${(chassis_length/2)-caster_wheel_radius}"/>
+	<xacro:property name="caster_wheel_origin_y" value="0.0"/>
 	<xacro:property name="caster_wheel_origin_z" value="${wheel_origin_z}"/>
 <!-- BASE LINK-->
@@ -40,5 +34,5 @@
 			<origin xyz="0 0 0" rpy="0 0 0"/>
 			<geometry>
-				<box size="${chassis_width} ${chassis_length} ${chassis_height}"/>
+				<box size="${chassis_length} ${chassis_width} ${chassis_height}"/>
 			</geometry>
 			<material name="orange"/>
@@ -47,8 +41,8 @@
 			<origin xyz="0 0 0" rpy="0 0 0"/>
 			<geometry>
-				<box size="${chassis_width} ${chassis_length} ${chassis_height}"/>
+				<box size="${chassis_length} ${chassis_width} ${chassis_height}"/>
 			</geometry>
 		</collision>
-		<xacro:inertial_box mass="${chassis_mass}" x="${chassis_width}" y="${chassis_length}" z="${chassis_height}">
+		<xacro:inertial_box mass="${chassis_mass}" x="${chassis_length}" y="${chassis_width}" z="${chassis_height}">
 			<origin xyz="0 0 0" rpy="0 0 0"/>
 		</xacro:inertial_box>
@@ -61,5 +55,5 @@
 		<parent link="chassis"/>
 		<child link="left_wheel"/>
-		<origin xyz="-${wheel_origin_x} ${wheel_origin_y} -${wheel_origin_z}" rpy="0 -${pi/2} 0"/>
+		<origin xyz="${wheel_origin_x} ${wheel_origin_y} -${wheel_origin_z}" rpy="-${pi/2} 0 0"/>
 		<axis xyz="0 0 1"/>
 	</joint>
@@ -73,5 +67,5 @@
 		<collision>
 			<geometry>
-				<cylinder radius="${wheel_radius}" length="${wheel_thickness}"/>
+				<sphere radius="${wheel_radius}"/>
 			</geometry>
 		</collision>
@@ -87,5 +81,5 @@
 		<parent link="chassis"/>
 		<child link="right_wheel"/>
-		<origin xyz="${wheel_origin_x} ${wheel_origin_y} -${wheel_origin_z}" rpy="0 ${pi/2} 0"/>
+		<origin xyz="${wheel_origin_x} -${wheel_origin_y} -${wheel_origin_z}" rpy="${pi/2} 0 0"/>
 		<axis xyz="0 0 -1"/>
 	</joint>
@@ -99,5 +93,5 @@
 		<collision>
 			<geometry>
-				<cylinder length="${wheel_thickness}" radius="${wheel_radius}"/>
+				<sphere radius="${wheel_radius}"/>
 			</geometry>
 		</collision>
@@ -141,5 +135,5 @@
 		<parent link="chassis"/>
 		<child link="back_caster_wheel"/>
-		<origin xyz="${caster_wheel_origin_x} -${caster_wheel_origin_y} -${caster_wheel_origin_z}" rpy="0 0 0"/>
+		<origin xyz="-${caster_wheel_origin_x} ${caster_wheel_origin_y} -${caster_wheel_origin_z}" rpy="0 0 0"/>
 		<!-- <axis xyz="1 1 0"/> -->
 	</joint>

Commit message: failed caster wheel

File: description/robot_core.xacro (robot description, xacro)
@@ -16,9 +16,15 @@
 	<xacro:property name="wheel_origin_y" value="${(chassis_width/2) + (wheel_thickness/2)}"/>
 	<xacro:property name="wheel_origin_z" value="${chassis_height/2}"/>
-    <xacro:property name="caster_wheel_radius" value="${wheel_radius}"/>
+	<xacro:property name="caster_dock_radius" value="0.05"/>
+	<xacro:property name="caster_dock_mass" value="0.1"/>
+	<xacro:property name="caster_dock_origin_x" value ="${(chassis_length/2)-caster_dock_radius}"/>
+	<xacro:property name="caster_dock_origin_y" value ="0.0"/>
+	<xacro:property name="caster_dock_origin_z" value ="${wheel_origin_z - wheel_radius}"/>
+    <xacro:property name="caster_wheel_radius" value="0.02"/>
+	<xacro:property name="caster_wheel_thickness" value="0.03"/>
     <xacro:property name="caster_wheel_mass" value="0.01"/>
-	<xacro:property name="caster_wheel_origin_x" value="${(chassis_length/2)-caster_wheel_radius}"/>
+	<xacro:property name="caster_wheel_origin_x" value="${caster_dock_radius}"/>
 	<xacro:property name="caster_wheel_origin_y" value="0.0"/>
-	<xacro:property name="caster_wheel_origin_z" value="${wheel_origin_z}"/>
+	<xacro:property name="caster_wheel_origin_z" value="${(wheel_radius * 2) - caster_wheel_radius}"/>
 	<xacro:property name="mu" value="0.001"/>
 <!-- BASE LINK-->
@@ -113,14 +119,35 @@
 	</gazebo>
 <!-- FRONT CASTER WHEEL-->
-	<joint name="front_caster_wheel_joint" type="fixed">
-		<parent link="chassis"/>
+	<joint name="front_caster_dock_joint" type="continuous">
+		<parent link="chassis"/>
+		<child link="front_caster_dock"/>
+		<origin xyz="${caster_dock_origin_x} ${caster_dock_origin_y} -${caster_dock_origin_z}" rpy="0 0 0"/>
+		<axis xyz="0 0 1"/>
+	</joint>
+	<link name="front_caster_dock">
+		<visual>
+			<geometry>
+				<cylinder radius="${caster_dock_radius}" length="0.0"/>
+			</geometry>
+		<material name="white"/>
+		</visual>
+		<collision>
+			<geometry>
+				<cylinder radius="${caster_dock_radius}" length="0.0"/>
+			</geometry>
+		</collision>
+		<xacro:inertial_cylinder mass="${caster_dock_mass}" length="0.0" radius="${caster_dock_radius}">
+			<origin xyz="0 0 0" rpy="0 0 0"/>
+		</xacro:inertial_cylinder>
+	</link>
+	<!-- <joint name="front_caster_wheel_joint" type="continuous">
+		<parent link="front_caster_dock"/>
 		<child link="front_caster_wheel"/>
-		<origin xyz="${caster_wheel_origin_x} ${caster_wheel_origin_y} -${caster_wheel_origin_z}" rpy="0 0 0"/>
-		<!-- <axis xyz="1 1 0"/> -->
+		<origin xyz="-${caster_wheel_origin_x} ${caster_wheel_origin_y} -${caster_wheel_origin_z}" rpy="${pi/2} 0 0"/>
 	</joint>
 	<link name="front_caster_wheel">
 		<visual>
 			<geometry>
-				<sphere radius="${caster_wheel_radius}"/>
+				<cylinder radius="${caster_wheel_radius}" length="${caster_wheel_thickness}"/>
 			</geometry>
 			<material name="white"/>
@@ -128,10 +155,10 @@
 		<collision>
 			<geometry>
-				<sphere radius="${caster_wheel_radius}"/>
-			</geometry>
-		</collision>
-		<xacro:inertial_sphere mass="${caster_wheel_mass}" radius="${caster_wheel_radius}">
-			<origin xyz="0 0 0" rpy="0 0 0"/>
-		</xacro:inertial_sphere>
+				<cylinder radius="${caster_wheel_radius}" length="${caster_wheel_thickness}"/>
+			</geometry>
+		</collision>
+		<xacro:inertial_cylinder mass="${caster_wheel_mass}" radius="${caster_wheel_radius}" length="${caster_wheel_thickness}">
+			<origin xyz="0 0 0" rpy="0 0 0"/>
+		</xacro:inertial_cylinder>
 	</link>
 	<gazebo reference="front_caster_wheel">
@@ -139,11 +166,11 @@
 		<mu1 value="${mu}"/>
 		<mu2 value="${mu}"/>
-	</gazebo>
+	</gazebo> -->
 <!-- BACK CASTER WHEEL-->
-	<joint name="back_caster_wheel_joint" type="fixed">
+	<!-- <joint name="back_caster_wheel_joint" type="fixed">
 		<parent link="chassis"/>
 		<child link="back_caster_wheel"/>
 		<origin xyz="-${caster_wheel_origin_x} ${caster_wheel_origin_y} -${caster_wheel_origin_z}" rpy="0 0 0"/>
-		<!-- <axis xyz="1 1 0"/> -->
+		<axis xyz="1 1 0"/>
 	</joint>
 	<link name="back_caster_wheel">
@@ -167,5 +194,5 @@
 		<mu1 value="${mu}"/>
 		<mu2 value="${mu}"/>
-	</gazebo>
+	</gazebo>	 -->
 	<joint name="back_frame_joint" type="fixed">
 		<parent link="chassis"/>
