Commit message: add xacro property

File: description/lidar.xacro (robot description, xacro)
@@ -4,7 +4,7 @@
 	<xacro:include filename="colours.xacro"/> -->
 	<joint name="laser_joint" type="fixed">
-		<parent link="chassis"/>
+		<parent link="front_caster_wheel"/>
 		<child link="laser_frame"/>
-		<origin xyz="0 0.122 0.212"/>
+		<origin xyz="0 0 ${chassis_height + 0.01}"/>
 	</joint>
 	<link name="laser_frame">
@@ -16,5 +16,5 @@
 		</visual>
 		<visual>
-            <origin xyz="0 0 -0.05"/>
+            <origin xyz="0 0 0"/>
             <geometry>
                 <cylinder radius="0.01" length="0.1"/>

File: description/robot_core.xacro (robot description, xacro)
@@ -3,4 +3,28 @@
 	<xacro:include filename="colours.xacro"/>
 	<xacro:include filename="inertial_macros.xacro"/>
+    <xacro:property name="chassis_length" value="0.3"/>
+    <xacro:property name="chassis_width" value="0.2"/>
+    <xacro:property name="chassis_height" value="0.11"/>
+    <xacro:property name="chassis_mass" value="1.0"/>
+	<xacro:property name="chassis_origin_x" value="0.0"/>
+	<xacro:property name="chassis_origin_y" value="${(chassis_length/2) + 0.05}"/>
+	<xacro:property name="chassis_origin_z" value="${(chassis_height/2 + wheel_radius)}"/>
+    <xacro:property name="wheel_radius" value="0.03"/>
+    <xacro:property name="wheel_thickness" value="0.03"/>
+    <xacro:property name="wheel_mass" value="0.05"/>
+    <xacro:property name="wheel_offset_x" value="0.0"/>
+    <xacro:property name="wheel_offset_y" value="0.0"/>
+    <xacro:property name="wheel_offset_z" value="0.0"/>
+	<xacro:property name="wheel_origin_x" value="${(chassis_width/2) + (wheel_thickness/2) + 0.01}"/>
+	<xacro:property name="wheel_origin_y" value="0.0"/>
+	<xacro:property name="wheel_origin_z" value="${chassis_height/2}"/>
+    <xacro:property name="caster_wheel_radius" value="${wheel_radius}"/>
+    <xacro:property name="caster_wheel_mass" value="0.01"/>
+	<xacro:property name="caster_wheel_offset_x" value="0.0"/>
+    <xacro:property name="caster_wheel_offset_y" value="0.0"/>
+    <xacro:property name="caster_wheel_offset_z" value="0.0"/>
+	<xacro:property name="caster_wheel_origin_x" value="0.0"/>
+	<xacro:property name="caster_wheel_origin_y" value="${(chassis_length/2)-caster_wheel_radius}"/>
+	<xacro:property name="caster_wheel_origin_z" value="${wheel_origin_z}"/>
 <!-- BASE LINK-->
 	<link name="base_link">
@@ -9,33 +33,33 @@
 		<parent link="base_link"/>
 		<child link="chassis"/>
-		<origin xyz="0 0.1 0"/>
+		<origin xyz="${chassis_origin_x} ${chassis_origin_y} ${chassis_origin_z}"/>
 	</joint>
 <!-- CHASSIS-->
 	<link name="chassis">
 		<visual>
-			<origin xyz="0 0.05 0.075" rpy="0 0 0"/>
+			<origin xyz="0 0 0" rpy="0 0 0"/>
 			<geometry>
-				<box size="0.3 0.3 0.15"/>
+				<box size="${chassis_width} ${chassis_length} ${chassis_height}"/>
 			</geometry>
-			<material name="white"/>
+			<material name="orange"/>
 		</visual>
 		<collision>
-			<origin xyz="0 0.05 0.075" rpy="0 0 0"/>
+			<origin xyz="0 0 0" rpy="0 0 0"/>
 			<geometry>
-				<box size="0.3 0.3 0.15"/>
+				<box size="${chassis_width} ${chassis_length} ${chassis_height}"/>
 			</geometry>
 		</collision>
-		<xacro:inertial_box mass="0.5" x="0.3" y="0.3" z="0.15">
-			<origin xyz="0 0.05 0.075" rpy="0 0 0"/>
+		<xacro:inertial_box mass="${chassis_mass}" x="${chassis_width}" y="${chassis_length}" z="${chassis_height}">
+			<origin xyz="0 0 0" rpy="0 0 0"/>
 		</xacro:inertial_box>
 	</link>
 	<gazebo reference="chassis">
-		<material>Gazebo/White</material>
+		<material>Gazebo/Orange</material>
 	</gazebo>
 <!-- LEFT WHEEL-->
 	<joint name="left_wheel_joint" type="continuous">
-		<parent link="base_link"/>
+		<parent link="chassis"/>
 		<child link="left_wheel"/>
-		<origin xyz="-0.175 0.05 0" rpy="0 -${pi/2} 0"/>
+		<origin xyz="-${wheel_origin_x} ${wheel_origin_y} -${wheel_origin_z}" rpy="0 -${pi/2} 0"/>
 		<axis xyz="0 0 1"/>
 	</joint>
@@ -43,5 +67,5 @@
 		<visual>
 			<geometry>
-				<cylinder radius="0.04" length="0.05"/>
+				<cylinder radius="${wheel_radius}" length="${wheel_thickness}"/>
 			</geometry>
 			<material name="blue"/>
@@ -49,8 +73,8 @@
 		<collision>
 			<geometry>
-				<cylinder radius="0.04" length="0.05"/>
+				<cylinder radius="${wheel_radius}" length="${wheel_thickness}"/>
 			</geometry>
 		</collision>
-		<xacro:inertial_cylinder mass="0.1" length="0.05" radius="0.05">
+		<xacro:inertial_cylinder mass="${wheel_mass}" length="${wheel_thickness}" radius="${wheel_radius}">
 			<origin xyz= "0 0 0" rpy="0 0 0"/>
 		</xacro:inertial_cylinder>
@@ -61,7 +85,7 @@
 <!-- RIGHT WHEEL-->
 	<joint name="right_wheel_joint" type="continuous">
-		<parent link="base_link"/>
+		<parent link="chassis"/>
 		<child link="right_wheel"/>
-		<origin xyz="0.175 0.05 0" rpy="0 ${pi/2} 0"/>
+		<origin xyz="${wheel_origin_x} ${wheel_origin_y} -${wheel_origin_z}" rpy="0 ${pi/2} 0"/>
 		<axis xyz="0 0 -1"/>
 	</joint>
@@ -69,5 +93,5 @@
 		<visual>
 			<geometry>
-				<cylinder length="0.04" radius="0.05"/>
+				<cylinder length="${wheel_thickness}" radius="${wheel_radius}"/>
 			</geometry>
 			<material name="blue"/>
@@ -75,8 +99,8 @@
 		<collision>
 			<geometry>
-				<cylinder length="0.04" radius="0.05"/>
+				<cylinder length="${wheel_thickness}" radius="${wheel_radius}"/>
 			</geometry>
 		</collision>
-		<xacro:inertial_cylinder mass="0.1" length="0.05" radius="0.05">
+		<xacro:inertial_cylinder mass="${wheel_mass}" length="${wheel_thickness}" radius="${wheel_radius}">
 			<origin xyz="0 0 0" rpy="0 0 0"/>
 		</xacro:inertial_cylinder>
@@ -85,29 +109,57 @@
 		<material>Gazebo/Blue</material>
 	</gazebo>
-<!-- CASTER WHEEL-->
-	<joint name="caster_wheel_joint" type="fixed">
+<!-- FRONT CASTER WHEEL-->
+	<joint name="front_caster_wheel_joint" type="fixed">
 		<parent link="chassis"/>
-		<child link="caster_wheel"/>
-		<origin xyz="0 0.15 0" rpy="0 0 0"/>
+		<child link="front_caster_wheel"/>
+		<origin xyz="${caster_wheel_origin_x} ${caster_wheel_origin_y} -${caster_wheel_origin_z}" rpy="0 0 0"/>
 		<!-- <axis xyz="1 1 0"/> -->
 	</joint>
-	<link name="caster_wheel">
+	<link name="front_caster_wheel">
 		<visual>
 			<geometry>
-				<sphere radius="0.05"/>
+				<sphere radius="${caster_wheel_radius}"/>
 			</geometry>
-			<material name="black"/>
+			<material name="white"/>
 		</visual>
 		<collision>
 			<geometry>
-				<sphere radius="0.05"/>
+				<sphere radius="${caster_wheel_radius}"/>
 			</geometry>
 		</collision>
-		<xacro:inertial_sphere mass="0.1" radius="0.05">
+		<xacro:inertial_sphere mass="${caster_wheel_mass}" radius="${caster_wheel_radius}">
 			<origin xyz="0 0 0" rpy="0 0 0"/>
 		</xacro:inertial_sphere>
 	</link>
-	<gazebo reference="caster_wheel">
-		<material>Gazebo/Black</material>
+	<gazebo reference="front_caster_wheel">
+		<material>Gazebo/White</material>
+		<mu1 value="0.001"/>
+		<mu2 value="0.001"/>
+	</gazebo>
+<!-- BACK CASTER WHEEL-->
+	<joint name="back_caster_wheel_joint" type="fixed">
+		<parent link="chassis"/>
+		<child link="back_caster_wheel"/>
+		<origin xyz="${caster_wheel_origin_x} -${caster_wheel_origin_y} -${caster_wheel_origin_z}" rpy="0 0 0"/>
+		<!-- <axis xyz="1 1 0"/> -->
+	</joint>
+	<link name="back_caster_wheel">
+		<visual>
+			<geometry>
+				<sphere radius="${caster_wheel_radius}"/>
+			</geometry>
+			<material name="white"/>
+		</visual>
+		<collision>
+			<geometry>
+				<sphere radius="${caster_wheel_radius}"/>
+			</geometry>
+		</collision>
+		<xacro:inertial_sphere mass="${caster_wheel_mass}" radius="${caster_wheel_radius}">
+			<origin xyz="0 0 0" rpy="0 0 0"/>
+		</xacro:inertial_sphere>
+	</link>
+	<gazebo reference="back_caster_wheel">
+		<material>Gazebo/White</material>
 		<mu1 value="0.001"/>
 		<mu2 value="0.001"/>

Commit message: rotation shim not triggered

File: description/lidar.xacro (robot description, xacro)
@@ -41,6 +41,6 @@
 					<horizontal>
 						<samples>360</samples>
-						<min_angle>-3.14</min_angle>
-						<max_angle>3.14</max_angle>
+						<min_angle>-1.57</min_angle>
+						<max_angle>1.57</max_angle>
 					</horizontal>
 				</scan>

File: description/robot_core.xacro (robot description, xacro)
@@ -16,15 +16,9 @@
 	<xacro:property name="wheel_origin_y" value="${(chassis_width/2) + (wheel_thickness/2)}"/>
 	<xacro:property name="wheel_origin_z" value="${chassis_height/2}"/>
-	<xacro:property name="caster_dock_radius" value="0.05"/>
-	<xacro:property name="caster_dock_mass" value="0.1"/>
-	<xacro:property name="caster_dock_origin_x" value ="${(chassis_length/2)-caster_dock_radius}"/>
-	<xacro:property name="caster_dock_origin_y" value ="0.0"/>
-	<xacro:property name="caster_dock_origin_z" value ="${wheel_origin_z - wheel_radius}"/>
-    <xacro:property name="caster_wheel_radius" value="0.02"/>
-	<xacro:property name="caster_wheel_thickness" value="0.03"/>
+    <xacro:property name="caster_wheel_radius" value="${wheel_radius}"/>
     <xacro:property name="caster_wheel_mass" value="0.01"/>
-	<xacro:property name="caster_wheel_origin_x" value="${caster_dock_radius}"/>
+	<xacro:property name="caster_wheel_origin_x" value="${(chassis_length/2)-caster_wheel_radius}"/>
 	<xacro:property name="caster_wheel_origin_y" value="0.0"/>
-	<xacro:property name="caster_wheel_origin_z" value="${(wheel_radius * 2) - caster_wheel_radius}"/>
+	<xacro:property name="caster_wheel_origin_z" value="${wheel_origin_z}"/>
 	<xacro:property name="mu" value="0.001"/>
 <!-- BASE LINK-->
@@ -119,35 +113,14 @@
 	</gazebo>
 <!-- FRONT CASTER WHEEL-->
-	<joint name="front_caster_dock_joint" type="continuous">
+	<joint name="front_caster_wheel_joint" type="fixed">
 		<parent link="chassis"/>
-		<child link="front_caster_dock"/>
-		<origin xyz="${caster_dock_origin_x} ${caster_dock_origin_y} -${caster_dock_origin_z}" rpy="0 0 0"/>
-		<axis xyz="0 0 1"/>
-	</joint>
-	<link name="front_caster_dock">
-		<visual>
-			<geometry>
-				<cylinder radius="${caster_dock_radius}" length="0.0"/>
-			</geometry>
-		<material name="white"/>
-		</visual>
-		<collision>
-			<geometry>
-				<cylinder radius="${caster_dock_radius}" length="0.0"/>
-			</geometry>
-		</collision>
-		<xacro:inertial_cylinder mass="${caster_dock_mass}" length="0.0" radius="${caster_dock_radius}">
-			<origin xyz="0 0 0" rpy="0 0 0"/>
-		</xacro:inertial_cylinder>
-	</link>
-	<!-- <joint name="front_caster_wheel_joint" type="continuous">
-		<parent link="front_caster_dock"/>
 		<child link="front_caster_wheel"/>
-		<origin xyz="-${caster_wheel_origin_x} ${caster_wheel_origin_y} -${caster_wheel_origin_z}" rpy="${pi/2} 0 0"/>
+		<origin xyz="${caster_wheel_origin_x} ${caster_wheel_origin_y} -${caster_wheel_origin_z}" rpy="0 0 0"/>
+		<!-- <axis xyz="1 1 0"/> -->
 	</joint>
 	<link name="front_caster_wheel">
 		<visual>
 			<geometry>
-				<cylinder radius="${caster_wheel_radius}" length="${caster_wheel_thickness}"/>
+				<sphere radius="${caster_wheel_radius}"/>
 			</geometry>
 			<material name="white"/>
@@ -155,10 +128,10 @@
 		<collision>
 			<geometry>
-				<cylinder radius="${caster_wheel_radius}" length="${caster_wheel_thickness}"/>
+				<sphere radius="${caster_wheel_radius}"/>
 			</geometry>
 		</collision>
-		<xacro:inertial_cylinder mass="${caster_wheel_mass}" radius="${caster_wheel_radius}" length="${caster_wheel_thickness}">
+		<xacro:inertial_sphere mass="${caster_wheel_mass}" radius="${caster_wheel_radius}">
 			<origin xyz="0 0 0" rpy="0 0 0"/>
-		</xacro:inertial_cylinder>
+		</xacro:inertial_sphere>
 	</link>
 	<gazebo reference="front_caster_wheel">
@@ -166,11 +139,11 @@
 		<mu1 value="${mu}"/>
 		<mu2 value="${mu}"/>
-	</gazebo> -->
+	</gazebo>
 <!-- BACK CASTER WHEEL-->
-	<!-- <joint name="back_caster_wheel_joint" type="fixed">
+	<joint name="back_caster_wheel_joint" type="fixed">
 		<parent link="chassis"/>
 		<child link="back_caster_wheel"/>
 		<origin xyz="-${caster_wheel_origin_x} ${caster_wheel_origin_y} -${caster_wheel_origin_z}" rpy="0 0 0"/>
-		<axis xyz="1 1 0"/>
+		<!-- <axis xyz="1 1 0"/> -->
 	</joint>
 	<link name="back_caster_wheel">
@@ -194,27 +167,4 @@
 		<mu1 value="${mu}"/>
 		<mu2 value="${mu}"/>
-	</gazebo>	 -->
-	<joint name="back_frame_joint" type="fixed">
-		<parent link="chassis"/>
-		<child link="back_frame"/>
-		<origin xyz="-${chassis_length/4} 0 ${chassis_height/2}" rpy="0 0 0"/>
-	</joint>
-	<link name="back_frame">
-		<visual>
-			<origin xyz="0 0 ${chassis_height/2}" rpy="0 0 0"/>
-			<geometry>
-				<box size="${chassis_length/2} ${chassis_width} ${chassis_height}"/>
-			</geometry>
-			<material name="orange"/>
-		</visual>
-		<collision>
-			<origin xyz="0 0 ${chassis_height/2}" rpy="0 0 0"/>
-			<geometry>
-				<box size="${chassis_length/2} ${chassis_width} ${chassis_height/2}"/>
-			</geometry>
-		</collision>
-		<xacro:inertial_box mass="${chassis_mass/2}" x="${chassis_length/2}" y="${chassis_width}" z="${chassis_height/2}">
-			<origin xyz="0 0 0" rpy="0 0 0"/>
-		</xacro:inertial_box>
-	</link>
+	</gazebo>
 </robot>

Commit message: final

File: description/lidar.xacro (robot description, xacro)
@@ -40,7 +40,7 @@
 				<scan>
 					<horizontal>
-						<samples>360</samples>
-						<min_angle>-3.14</min_angle>
-						<max_angle>3.14</max_angle>
+						<samples>190</samples>
+						<min_angle>-1.65</min_angle>
+						<max_angle>1.65</max_angle>
 					</horizontal>
 				</scan>

File: description/robot_core.xacro (robot description, xacro)
@@ -7,5 +7,5 @@
     <xacro:property name="chassis_height" value="0.2"/>
     <xacro:property name="chassis_mass" value="1.0"/>
-	<xacro:property name="chassis_origin_x" value="${(chassis_length/2) + 0.005}"/>
+	<xacro:property name="chassis_origin_x" value="${(chassis_length/2)}"/>
 	<xacro:property name="chassis_origin_y" value="0.0"/>
 	<xacro:property name="chassis_origin_z" value="${(chassis_height/2 + wheel_radius)}"/>
@@ -21,5 +21,5 @@
 	<xacro:property name="caster_wheel_origin_y" value="0.0"/>
 	<xacro:property name="caster_wheel_origin_z" value="${wheel_origin_z}"/>
-	<xacro:property name="mu" value="0.001"/>
+	<xacro:property name="mu" value="0.1"/>
 <!-- BASE LINK-->
 	<link name="base_link">

File: description/ros2_control.xacro (robot description, xacro)
@@ -35,6 +35,6 @@
 		<joint name="left_wheel_joint">
 			<command_interface name="velocity">
-				<param name="min">-10</param>
-				<param name="max">10</param>
+				<param name="min">-0.5</param>
+				<param name="max">0.5</param>
 			</command_interface>
 			<state_interface name="position"/>
@@ -43,6 +43,6 @@
 		<joint name="right_wheel_joint">
 			<command_interface name="velocity">
-				<param name="min">-10</param>
-				<param name="max">10</param>
+				<param name="min">-0.5</param>
+				<param name="max">0.5</param>
 			</command_interface>
 			<state_interface name="position"/>
